File: steno.kicad_pcb (KiCad board)
At the start: 2 copper layers, 75 parts, among them J1 USB_C_Receptacle_USB2.0_14P, SW1 SW_Push, U1 RP2040, U2 AP2127N-3.3, U3 W25Q16JVSS, Y1 12 MHz

Commit message: Savepoint!
Parts:
- D10, D11, D12, D13, D14, D15, D16, D17, D18, D19, D2, D20, D21, D22, D23, D24, D25, D26, D3, D4, D5, D6, D7, D8, D9: moved to B.Cu
- moved R4 167.1 mm to (48.4, 44.4), turned to -90 degrees
- moved R1 163.5 mm to (50.2, 44.4), turned to -90 degrees
- moved R2 162.7 mm to (51.8, 44.4), turned to -90 degrees
- moved R3 161.5 mm to (53.6, 44.4), turned to -90 degrees
- moved J1 160.6 mm to (51.0, 38.0), turned to 180 degrees
- moved C4 156.1 mm to (43.0, 45.0), turned to -90 degrees
- moved D1 151.3 mm to (61.5, 45.5), turned to 180 degrees
- moved D16 149.9 mm to (232.0, 60.1), turned to 90 degrees
- moved D21 149.9 mm to (232.0, 77.1), turned to 90 degrees
- moved D15 145.6 mm to (214.0, 60.1), turned to 90 degrees
- moved U2 143.4 mm to (75.5, 46.3), turned to 180 degrees
- moved C12 139.7 mm to (67.0, 46.3), turned to -90 degrees
- moved S25 135.7 mm to (173.0, 107.0), turned to 0 degrees
- moved C11 134.5 mm to (71.5, 46.3), turned to -90 degrees
- moved D20 131.6 mm to (214.0, 77.1), turned to 90 degrees
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Connections:
- D10 pad 1: COL_2 -> ROW_2
- D11 pad 1: COL_2 -> ROW_2
- D12 pad 1: COL_3 -> ROW_3
- D13 pad 1: COL_3 -> ROW_3
- D14 pad 1: COL_3 -> ROW_3
- D15 pad 1: COL_3 -> ROW_3
- D16 pad 1: COL_3 -> ROW_3
- D17 pad 1: COL_4 -> ROW_4
- D18 pad 1: COL_4 -> ROW_4
- D19 pad 1: COL_4 -> ROW_4
- D2 pad 1: COL_1 -> ROW_1
- D20 pad 1: COL_4 -> ROW_4
- D21 pad 1: COL_4 -> ROW_4
- D22 pad 1: COL_5 -> ROW_5
- D23 pad 1: COL_5 -> ROW_5
- D24 pad 1: COL_5 -> ROW_5
- D25 pad 1: COL_5 -> ROW_5
- D26 pad 1: COL_5 -> ROW_5
- D3 pad 1: COL_1 -> ROW_1
- D4 pad 1: COL_1 -> ROW_1
- D5 pad 1: COL_1 -> ROW_1
- D6 pad 1: COL_1 -> ROW_1
- D7 pad 1: COL_2 -> ROW_2
- D8 pad 1: COL_2 -> ROW_2
- D9 pad 1: COL_2 -> ROW_2
- U1 pad 14: COL_1 -> ROW_1
- U1 pad 15: COL_2 -> ROW_2
- U1 pad 16: COL_3 -> ROW_3
- U1 pad 17: COL_4 -> ROW_4
- U1 pad 18: COL_5 -> ROW_5
Routing:
- net +3.3V: track 0.00 -> 95.3 mm, vias 0 -> 2
- net D+: track 0.00 -> 92.4 mm, vias 0 -> 2
- net D-: track 0.00 -> 90.9 mm, vias 0 -> 2
- net ROW_1: track 0.00 -> 73.1 mm
- net ROW_4: track 0.00 -> 72.4 mm
- net ROW_3: track 0.00 -> 72.4 mm
- net ROW_2: track 0.00 -> 72.3 mm
- net GND: track 0.00 -> 63.6 mm, vias 0 -> 17
- net Net-(J1-SHIELD): track 0.00 -> 22.7 mm
- net COL_5: track 0.00 -> 17.0 mm, vias 0 -> 2
- net COL_4: track 0.00 -> 17.0 mm, vias 0 -> 2
- net COL_3: track 0.00 -> 17.0 mm, vias 0 -> 2
- net COL_2: track 0.00 -> 17.0 mm, vias 0 -> 2
- net COL_1: track 0.00 -> 17.0 mm
- net QSPI_SS: track 0.00 -> 15.9 mm
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- added copper zone on In2.Cu, net +3.3V
- added copper zone on In1.Cu, net GND
Other:
- copper layers 2 -> 4

Commit message: Savepoint!
Parts:
- moved S21 175.5 mm to (276.0, 93.5), turned to 90 degrees
- moved D22 168.8 mm to (277.1, 84.5), turned to 180 degrees
- moved S22 160.1 mm to (276.0, 75.5), turned to 90 degrees
- moved D23 154.9 mm to (277.1, 66.5), turned to 180 degrees
- moved S23 147.6 mm to (276.0, 57.5), turned to 90 degrees
- moved D24 144.1 mm to (277.1, 48.5), turned to 180 degrees
- moved S24 138.6 mm to (276.0, 39.5), turned to 90 degrees
- moved D25 137.2 mm to (277.1, 30.5), turned to 180 degrees
- moved D26 134.9 mm to (277.1, 12.5), turned to 180 degrees
- moved S25 133.9 mm to (276.0, 21.5), turned to 90 degrees
- moved C4 98.9 mm to (139.9, 64.7)
- moved J1 98.9 mm to (147.9, 57.7)
- moved R1 98.9 mm to (147.2, 64.2)
- moved R2 98.9 mm to (148.7, 64.2)
- moved R3 98.9 mm to (150.6, 64.2)
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Routing:
- net ROW_1: track 73.1 -> 0.00 mm
- net ROW_4: track 72.4 -> 0.00 mm
- net ROW_3: track 72.4 -> 0.00 mm
- net ROW_2: track 72.3 -> 0.00 mm
- net D+: track 92.4 -> 36.7 mm
- net D-: track 90.9 -> 35.9 mm
- net +3.3V: track 95.3 -> 52.1 mm, vias 2 -> 11
- net COL_5: track 17.0 -> 0.00 mm, vias 2 -> 0
- net COL_4: track 17.0 -> 0.00 mm, vias 2 -> 0
- net COL_3: track 17.0 -> 0.00 mm, vias 2 -> 0
- net COL_2: track 17.0 -> 0.00 mm, vias 2 -> 0
- net COL_1: track 17.0 -> 0.00 mm
- net GND: track 63.6 -> 53.0 mm, vias 17 -> 22
- net Net-(D8-A): track 3.51 -> 0.00 mm
- net Net-(D7-A): track 3.51 -> 0.00 mm
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Other:
- board outline added: 200.3 x 94.7 mm

Commit message: Savepoint!
Parts:
- removed D22, D23, D24, D25, D26: 1N914, Diode_SMD:D_SOD-123
- removed S21, S22, S23, S24, S25: Keyswitch, ScottoKeebs_Hotswap:Hotswap_Choc_V1V2_1.00u
- D1: footprint Diode_SMD:D_SOD-123 -> Diode_SMD:D_SOD-323F
- SW1: footprint Button_Switch_SMD:SW_SPST_TL3305A -> Button_Switch_THT:SW_PUSH_6mm
- moved SW1 5.49 mm to (153.2, 109.2)
- moved D21 4.29 mm to (170.1, 129.6)
- moved D16 4.16 mm to (191.2, 105.9)
- moved D12 4.15 mm to (191.2, 66.0)
- moved D14 4.15 mm to (227.2, 66.0)
- moved D15 4.15 mm to (245.2, 83.0)
- moved C1 4.11 mm to (146.0, 92.0)
- moved C10 4.11 mm to (155.9, 96.4)
- moved C11 4.11 mm to (153.8, 72.8)
- moved C12 4.11 mm to (153.8, 69.9)
- moved C13 4.11 mm to (145.6, 68.6)
- moved C2 4.11 mm to (143.7, 87.3)
- moved C3 4.11 mm to (150.0, 80.8)
- moved C5 4.11 mm to (143.1, 68.6)
- moved C6 4.11 mm to (143.7, 82.5)
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Connections:
- D12 pad 1: ROW_3 -> ROW_1
- D13 pad 1: ROW_3 -> ROW_1
- D14 pad 1: ROW_3 -> ROW_1
- D15 pad 1: ROW_3 -> ROW_1
- D16 pad 1: ROW_3 -> ROW_1
- D17 pad 1: ROW_4 -> ROW_2
- D18 pad 1: ROW_4 -> ROW_2
- D19 pad 1: ROW_4 -> ROW_2
- D20 pad 1: ROW_4 -> ROW_2
- D21 pad 1: ROW_4 -> ROW_2
- S11 pad 1: COL_1 -> COL_6
- S12 pad 1: COL_2 -> COL_7
- S13 pad 1: COL_3 -> COL_8
- S14 pad 1: COL_4 -> COL_9
- S15 pad 1: COL_5 -> COL_10
- S16 pad 1: COL_1 -> COL_6
- S17 pad 1: COL_2 -> COL_7
- S18 pad 1: COL_3 -> COL_8
- S19 pad 1: COL_4 -> COL_9
- S20 pad 1: COL_5 -> COL_10
- U1 pad 11: unconnected-(U1-GPIO8-Pad11) -> COL_8
- U1 pad 12: unconnected-(U1-GPIO9-Pad12) -> COL_9
- U1 pad 13: unconnected-(U1-GPIO10-Pad13) -> COL_10
- U1 pad 16: ROW_3 -> unconnected-(U1-GPIO13-Pad16)
- U1 pad 17: ROW_4 -> unconnected-(U1-GPIO14-Pad17)
- U1 pad 18: ROW_5 -> unconnected-(U1-GPIO15-Pad18)
- U1 pad 29: unconnected-(U1-GPIO18-Pad29) -> COL_3
- U1 pad 3: COL_1 -> unconnected-(U1-GPIO1-Pad3)
- U1 pad 36: unconnected-(U1-GPIO24-Pad36) -> COL_2
- U1 pad 37: unconnected-(U1-GPIO25-Pad37) -> COL_1
- U1 pad 4: COL_2 -> unconnected-(U1-GPIO2-Pad4)
- U1 pad 5: COL_3 -> unconnected-(U1-GPIO3-Pad5)
- U1 pad 8: unconnected-(U1-GPIO6-Pad8) -> COL_6
- U1 pad 9: unconnected-(U1-GPIO7-Pad9) -> COL_7
Routing:
- net ROW_1: track 0.00 -> 458.5 mm, vias 0 -> 5
- net ROW_2: track 0.00 -> 404.5 mm, vias 0 -> 5
- net COL_2: track 0.00 -> 118.5 mm, vias 0 -> 5
- net COL_1: track 0.00 -> 115.0 mm, vias 0 -> 3
- net COL_3: track 0.00 -> 114.2 mm, vias 0 -> 3
- net COL_9: track 0.00 -> 111.9 mm, vias 0 -> 3
- net COL_8: track 0.00 -> 101.5 mm, vias 0 -> 7
- net COL_7: track 0.00 -> 91.7 mm, vias 0 -> 3
- net COL_4: track 0.00 -> 81.5 mm, vias 0 -> 3
- net COL_5: track 0.00 -> 79.1 mm, vias 0 -> 3
- net COL_6: track 0.00 -> 68.9 mm, vias 0 -> 1
- net COL_10: track 0.00 -> 57.4 mm, vias 0 -> 3
- net Net-(D6-A): track 0.00 -> 3.63 mm
- net Net-(D13-A): track 0.00 -> 3.55 mm
- net Net-(D8-A): track 0.00 -> 3.51 mm
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- added copper zone on B.Cu, net (none)
- added copper zone on F.Cu, net (none)
