File: key_layout.kicad_sch (KiCad schematic)
At the start: 48 parts

Commit message: Fixing buttons / Transitioning to new computer.
Parts:
- renumbered D25 to D10, D4 to D11, D9 to D12, D14 to D13, D19 to D14, D24 to D15, D5 to D16, D10 to D17, D15 to D18, D20 to D19, D22 to D20, D6 to D21, D11 to D22, D16 to D23, D21 to D24, D23 to D25, D7 to D3, D12 to D4, D17 to D5, D3 to D6, D8 to D7, D13 to D8, D18 to D9
Changed lines of the file:
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@@
 		(dnp no)
 		(fields_autoplaced yes)
-		(property "Reference" "D16"
+		(property "Reference" "D23"
 			(at 90.17 83.8199 90)
 			(show_name no)
@@
 			(project "steno"
 				(path "/238e1d3b-9ec5-448b-85c7-386a29cd2631/194d9414-d5fd-4d49-94c7-ab8062ec2e41"
-					(reference "D16")
+					(reference "D23")
 					(unit 1)
 				)
@@
 		(dnp no)
 		(fields_autoplaced yes)
-		(property "Reference" "D7"
+		(property "Reference" "D3"
 			(at 39.37 64.7699 90)
 			(show_name no)
@@
 			(project "steno"
 				(path "/238e1d3b-9ec5-448b-85c7-386a29cd2631/194d9414-d5fd-4d49-94c7-ab8062ec2e41"
-					(reference "D7")
+					(reference "D3")
 					(unit 1)
 				)
@@
 		(dnp no)
 		(fields_autoplaced yes)
-		(property "Reference" "D10"
+		(property "Reference" "D17"
 			(at 77.47 64.7699 90)
 			(show_name no)
@@
 			(project "steno"
 				(path "/238e1d3b-9ec5-448b-85c7-386a29cd2631/194d9414-d5fd-4d49-94c7-ab8062ec2e41"
-					(reference "D10")
+					(reference "D17")
 					(unit 1)
 				)
@@
 		(dnp no)
 		(fields_autoplaced yes)
-		(property "Reference" "D20"
+		(property "Reference" "D19"
 			(at 77.47 102.8699 90)
 			(show_name no)
@@
 			(project "steno"
 				(path "/238e1d3b-9ec5-448b-85c7-386a29cd2631/194d9414-d5fd-4d49-94c7-ab8062ec2e41"
-					(reference "D20")
+					(reference "D19")
 					(unit 1)
 				)
@@
 		(dnp no)
 		(fields_autoplaced yes)
-		(property "Reference" "D13"
+		(property "Reference" "D8"
 			(at 52.07 83.8199 90)
 			(show_name no)
@@
 			(project "steno"
 				(path "/238e1d3b-9ec5-448b-85c7-386a29cd2631/194d9414-d5fd-4d49-94c7-ab8062ec2e41"
-					(reference "D13")
+					(reference "D8")
 					(unit 1)
 				)
@@
 		(dnp no)
 		(fields_autoplaced yes)
-		(property "Reference" "D18"
+		(property "Reference" "D9"
 			(at 52.07 102.8699 90)
 			(show_name no)
@@
 			(project "steno"
 				(path "/238e1d3b-9ec5-448b-85c7-386a29cd2631/194d9414-d5fd-4d49-94c7-ab8062ec2e41"
-					(reference "D18")
+					(reference "D9")
 					(unit 1)
 				)
@@
 		(dnp no)
 		(fields_autoplaced yes)
-		(property "Reference" "D3"
+		(property "Reference" "D6"
 			(at 52.07 45.7199 90)
 			(show_name no)
@@
 			(project "steno"
 				(path "/238e1d3b-9ec5-448b-85c7-386a29cd2631/194d9414-d5fd-4d49-94c7-ab8062ec2e41"
-					(reference "D3")
+					(reference "D6")
 					(unit 1)
 				)
@@
 		(dnp no)
 		(fields_autoplaced yes)
-		(property "Reference" "D17"
+		(property "Reference" "D5"
 			(at 39.37 102.8699 90)
 			(show_name no)
@@
 			(project "steno"
 				(path "/238e1d3b-9ec5-448b-85c7-386a29cd2631/194d9414-d5fd-4d49-94c7-ab8062ec2e41"
-					(reference "D17")
+					(reference "D5")
 					(unit 1)
 				)
@@
 		(dnp no)
 		(fields_autoplaced yes)
-		(property "Reference" "D15"
+		(property "Reference" "D18"
 			(at 77.47 83.8199 90)
 			(show_name no)
@@
 			(project "steno"
 				(path "/238e1d3b-9ec5-448b-85c7-386a29cd2631/194d9414-d5fd-4d49-94c7-ab8062ec2e41"
-					(reference "D15")
+					(reference "D18")
 					(unit 1)
 				)
@@
 		(dnp no)
 		(fields_autoplaced yes)
-		(property "Reference" "D5"
+		(property "Reference" "D16"
 			(at 77.47 45.7199 90)
 			(show_name no)
@@
 			(project "steno"
 				(path "/238e1d3b-9ec5-448b-85c7-386a29cd2631/194d9414-d5fd-4d49-94c7-ab8062ec2e41"
-					(reference "D5")
+					(reference "D16")
 					(unit 1)
 				)
@@
 		(dnp no)
 		(fields_autoplaced yes)
-		(property "Reference" "D19"
+		(property "Reference" "D14"
 			(at 64.77 102.8699 90)
 			(show_name no)
@@
 			(project "steno"
 				(path "/238e1d3b-9ec5-448b-85c7-386a29cd2631/194d9414-d5fd-4d49-94c7-ab8062ec2e41"
-					(reference "D19")
+					(reference "D14")
 					(unit 1)
 				)
@@
 		(dnp no)
 		(fields_autoplaced yes)
-		(property "Reference" "D12"
+		(property "Reference" "D4"
 			(at 39.37 83.8199 90)
 			(show_name no)
@@
 			(project "steno"
 				(path "/238e1d3b-9ec5-448b-85c7-386a29cd2631/194d9414-d5fd-4d49-94c7-ab8062ec2e41"
-					(reference "D12")
+					(reference "D4")
 					(unit 1)
 				)
@@
 		(dnp no)
 		(fields_autoplaced yes)
-		(property "Reference" "D4"
+		(property "Reference" "D11"
 			(at 64.77 45.7199 90)
 			(show_name no)
@@
 			(project "steno"
 				(path "/238e1d3b-9ec5-448b-85c7-386a29cd2631/194d9414-d5fd-4d49-94c7-ab8062ec2e41"
-					(reference "D4")
+					(reference "D11")
 					(unit 1)
 				)
@@
 		(dnp no)
 		(fields_autoplaced yes)
-		(property "Reference" "D14"
+		(property "Reference" "D13"
 			(at 64.77 83.8199 90)
 			(show_name no)
@@
 			(project "steno"
 				(path "/238e1d3b-9ec5-448b-85c7-386a29cd2631/194d9414-d5fd-4d49-94c7-ab8062ec2e41"
-					(reference "D14")
+					(reference "D13")
 					(unit 1)
 				)
@@
 		(in_pos_files yes)
 		(dnp no)
-		(property "Reference" "D11"
+		(property "Reference" "D22"
 			(at 90.17 64.7699 90)
 			(show_name no)
@@
 			(project "steno"
 				(path "/238e1d3b-9ec5-448b-85c7-386a29cd2631/194d9414-d5fd-4d49-94c7-ab8062ec2e41"
-					(reference "D11")
+					(reference "D22")
 					(unit 1)
 				)
@@
 		(dnp no)
 		(fields_autoplaced yes)
-		(property "Reference" "D22"
+		(property "Reference" "D20"
 			(at 77.47 121.9199 90)
 			(show_name no)
@@
 			(project "steno"
 				(path "/238e1d3b-9ec5-448b-85c7-386a29cd2631/194d9414-d5fd-4d49-94c7-ab8062ec2e41"
-					(reference "D22")
+					(reference "D20")
 					(unit 1)
 				)
@@
 		(dnp no)
 		(fields_autoplaced yes)
-		(property "Reference" "D21"
+		(property "Reference" "D24"
 			(at 90.17 102.8699 90)
 			(show_name no)
@@
 			(project "steno"
 				(path "/238e1d3b-9ec5-448b-85c7-386a29cd2631/194d9414-d5fd-4d49-94c7-ab8062ec2e41"
-					(reference "D21")
+					(reference "D24")
 					(unit 1)
 				)
@@
 		(dnp no)
 		(fields_autoplaced yes)
-		(property "Reference" "D8"
+		(property "Reference" "D7"
 			(at 52.07 64.7699 90)
 			(show_name no)
@@
 			(project "steno"
 				(path "/238e1d3b-9ec5-448b-85c7-386a29cd2631/194d9414-d5fd-4d49-94c7-ab8062ec2e41"
-					(reference "D8")
+					(reference "D7")
 					(unit 1)
 				)
@@
 		(dnp no)
 		(fields_autoplaced yes)
-		(property "Reference" "D6"
+		(property "Reference" "D21"
 			(at 90.17 45.7199 90)
 			(show_name no)
@@
 			(project "steno"
 				(path "/238e1d3b-9ec5-448b-85c7-386a29cd2631/194d9414-d5fd-4d49-94c7-ab8062ec2e41"
-					(reference "D6")
+					(reference "D21")
 					(unit 1)
 				)
@@
 		(dnp no)
 		(fields_autoplaced yes)
-		(property "Reference" "D9"
+		(property "Reference" "D12"
 			(at 64.77 64.7699 90)
 			(show_name no)
@@
 			(project "steno"
 				(path "/238e1d3b-9ec5-448b-85c7-386a29cd2631/194d9414-d5fd-4d49-94c7-ab8062ec2e41"
-					(reference "D9")
+					(reference "D12")
 					(unit 1)
 				)
@@
 		(dnp no)
 		(fields_autoplaced yes)
-		(property "Reference" "D24"
+		(property "Reference" "D15"
 			(at 64.77 121.9199 90)
 			(show_name no)
@@
 			(project "steno"
 				(path "/238e1d3b-9ec5-448b-85c7-386a29cd2631/194d9414-d5fd-4d49-94c7-ab8062ec2e41"
-					(reference "D24")
+					(reference "D15")
 					(unit 1)
 				)
@@
 		(dnp no)
 		(fields_autoplaced yes)
-		(property "Reference" "D25"
+		(property "Reference" "D10"
 			(at 52.07 121.9199 90)
 			(show_name no)
@@
 			(project "steno"
 				(path "/238e1d3b-9ec5-448b-85c7-386a29cd2631/194d9414-d5fd-4d49-94c7-ab8062ec2e41"
-					(reference "D25")
+					(reference "D10")
 					(unit 1)
 				)
@@
 		(dnp no)
 		(fields_autoplaced yes)
-		(property "Reference" "D23"
+		(property "Reference" "D25"
 			(at 90.17 121.9199 90)
 			(show_name no)
@@
 			(project "steno"
 				(path "/238e1d3b-9ec5-448b-85c7-386a29cd2631/194d9414-d5fd-4d49-94c7-ab8062ec2e41"
-					(reference "D23")
+					(reference "D25")
 					(unit 1)
 				)

Commit message: Init Commit!
Parts:
- added SW1: Switch, Button_Switch_SMD:SW_SPST_PTS810, symbol ScottoKeebs:Placeholder_Switch
- added U2: RP2040_Pro_Micro, 3rd_party_footprints:RP2040_Pro_Micro, symbol 3rd_party_symbols:rp2040_pro_micro
Connections:
- net COL_1: now also U2.24 (gp21)
- net COL_2: now also U2.23 (gp23)
- net COL_3: now also U2.22 (gp20)
- net COL_4: now also U2.21 (gp22)
- net COL_5: now also U2.20 (gp26)
- net ROW_1: now also U2.10 (gp7)
- net ROW_2: now also U2.11 (gp8)
- net ROW_3: now also U2.18 (gp28)
- net ROW_4: now also U2.19 (gp27)
- net ROW_5: now also U2.12 (gp9)
- new net: SW1.1, U2.15 (RST)
- new net GND: SW1.2, U2.14 (GND), U2.3 (GND), U2.4 (GND)
